File: sch/A-DSP V10.sch (EAGLE design)
At the start: 96 parts, among them CON2 350760-4, CON3 350760-4, CON4 794681-8, IC4 317T, IC6 DSPIC33FJXXXGP802SMT, Q1 IRF530, Q2. IRF530, Q3 IRF530, Q4 IRF530, U3 HIP4081AIBZ

Commit message: Add files via upload
Parts:
- R17, R20, R25, R27: value 5R -> 22R
- R18, R21, R24, R28: value 5R -> 47R
Connections:
- removed net N$17: R17.2, R18.1
- removed net N$4: Q3.G, R25.2
- new net N$67: R17.2
- net N$10: now also R25.1
- net N$11: now also R18.1
- net N$48: now also R25.2; no longer R27.1, R28.2
- net N$6: now also R28.2; no longer R27.2
- net N$61: now also Q3.G; no longer R25.1
- net N$62: now also R27.2; no longer R20.2, R21.2
- net N$63: now also R21.2
- net N$8: now also R27.1
Other:
- note added: "1N4148"
- note added: "D4"
- note added: "D5"
- note added: "D6"
- note added: "D7"
- moved on the sheet: R17, R18, R20, R21, R24, R25, R27, R28
